Commit message: rename robot 1 and 2

File: src/moveit_control/fairino_dual_moveit_config/config/fairino.ros2_control.real.xacro (robot description, xacro)
@@ -7,4 +7,45 @@
                 <!-- By default, set up controllers for simulation. This won't work on real hardware -->
                 <plugin>fairino_hardware/FairinoHardwareInterface</plugin>
+            </hardware>
+            <joint name="robot2_j1">
+                <command_interface name="position"/>
+                <state_interface name="position">
+                  <param name="initial_value">${initial_positions['robot2_j1']}</param>
+                </state_interface>
+            </joint>
+            <joint name="robot2_j2">
+                <command_interface name="position"/>
+                <state_interface name="position">
+                  <param name="initial_value">${initial_positions['robot2_j2']}</param>
+                </state_interface>
+            </joint>
+            <joint name="robot2_j3">
+                <command_interface name="position"/>
+                <state_interface name="position">
+                  <param name="initial_value">${initial_positions['robot2_j3']}</param>
+                </state_interface>
+            </joint>
+            <joint name="robot2_j4">
+                <command_interface name="position"/>
+                <state_interface name="position">
+                  <param name="initial_value">${initial_positions['robot2_j4']}</param>
+                </state_interface>
+            </joint>
+            <joint name="robot2_j5">
+                <command_interface name="position"/>
+                <state_interface name="position">
+                  <param name="initial_value">${initial_positions['robot2_j5']}</param>
+                </state_interface>
+            </joint>
+            <joint name="robot2_j6">
+                <command_interface name="position"/>
+                <state_interface name="position">
+                  <param name="initial_value">${initial_positions['robot2_j6']}</param>
+                </state_interface>
+            </joint>
+        </ros2_control>
+        <ros2_control name="${name2}" type="system">
+            <hardware>
+                <plugin>fairino_hardware/FairinoHardwareInterface2</plugin>
             </hardware>
             <joint name="robot1_j1">
@@ -45,45 +86,4 @@
             </joint>
         </ros2_control>
-        <ros2_control name="${name2}" type="system">
-            <hardware>
-                <plugin>fairino_hardware/FairinoHardwareInterface2</plugin>
-            </hardware>
-            <joint name="robot2_j1">
-                <command_interface name="position"/>
-                <state_interface name="position">
-                  <param name="initial_value">${initial_positions['robot2_j1']}</param>
-                </state_interface>
-            </joint>
-            <joint name="robot2_j2">
-                <command_interface name="position"/>
-                <state_interface name="position">
-                  <param name="initial_value">${initial_positions['robot2_j2']}</param>
-                </state_interface>
-            </joint>
-            <joint name="robot2_j3">
-                <command_interface name="position"/>
-                <state_interface name="position">
-                  <param name="initial_value">${initial_positions['robot2_j3']}</param>
-                </state_interface>
-            </joint>
-            <joint name="robot2_j4">
-                <command_interface name="position"/>
-                <state_interface name="position">
-                  <param name="initial_value">${initial_positions['robot2_j4']}</param>
-                </state_interface>
-            </joint>
-            <joint name="robot2_j5">
-                <command_interface name="position"/>
-                <state_interface name="position">
-                  <param name="initial_value">${initial_positions['robot2_j5']}</param>
-                </state_interface>
-            </joint>
-            <joint name="robot2_j6">
-                <command_interface name="position"/>
-                <state_interface name="position">
-                  <param name="initial_value">${initial_positions['robot2_j6']}</param>
-                </state_interface>
-            </joint>
-        </ros2_control>
     </xacro:macro>
 </robot>

File: src/moveit_control/fairino_dual_moveit_config/config/fairino.ros2_control.xacro (robot description, xacro)
@@ -8,4 +8,40 @@
                 <plugin>mock_components/GenericSystem</plugin>
             </hardware>
+            <joint name="robot2_j1">
+                <command_interface name="position"/>
+                <state_interface name="position">
+                  <param name="initial_value">${initial_positions['robot2_j1']}</param>
+                </state_interface>
+            </joint>
+            <joint name="robot2_j2">
+                <command_interface name="position"/>
+                <state_interface name="position">
+                  <param name="initial_value">${initial_positions['robot2_j2']}</param>
+                </state_interface>
+            </joint>
+            <joint name="robot2_j3">
+                <command_interface name="position"/>
+                <state_interface name="position">
+                  <param name="initial_value">${initial_positions['robot2_j3']}</param>
+                </state_interface>
+            </joint>
+            <joint name="robot2_j4">
+                <command_interface name="position"/>
+                <state_interface name="position">
+                  <param name="initial_value">${initial_positions['robot2_j4']}</param>
+                </state_interface>
+            </joint>
+            <joint name="robot2_j5">
+                <command_interface name="position"/>
+                <state_interface name="position">
+                  <param name="initial_value">${initial_positions['robot2_j5']}</param>
+                </state_interface>
+            </joint>
+            <joint name="robot2_j6">
+                <command_interface name="position"/>
+                <state_interface name="position">
+                  <param name="initial_value">${initial_positions['robot2_j6']}</param>
+                </state_interface>
+            </joint>
             <joint name="robot1_j1">
                 <command_interface name="position"/>
@@ -44,40 +80,4 @@
                 </state_interface>
             </joint>
-            <joint name="robot2_j1">
-                <command_interface name="position"/>
-                <state_interface name="position">
-                  <param name="initial_value">${initial_positions['robot2_j1']}</param>
-                </state_interface>
-            </joint>
-            <joint name="robot2_j2">
-                <command_interface name="position"/>
-                <state_interface name="position">
-                  <param name="initial_value">${initial_positions['robot2_j2']}</param>
-                </state_interface>
-            </joint>
-            <joint name="robot2_j3">
-                <command_interface name="position"/>
-                <state_interface name="position">
-                  <param name="initial_value">${initial_positions['robot2_j3']}</param>
-                </state_interface>
-            </joint>
-            <joint name="robot2_j4">
-                <command_interface name="position"/>
-                <state_interface name="position">
-                  <param name="initial_value">${initial_positions['robot2_j4']}</param>
-                </state_interface>
-            </joint>
-            <joint name="robot2_j5">
-                <command_interface name="position"/>
-                <state_interface name="position">
-                  <param name="initial_value">${initial_positions['robot2_j5']}</param>
-                </state_interface>
-            </joint>
-            <joint name="robot2_j6">
-                <command_interface name="position"/>
-                <state_interface name="position">
-                  <param name="initial_value">${initial_positions['robot2_j6']}</param>
-                </state_interface>
-            </joint>
         </ros2_control>
     </xacro:macro>

File: src/moveit_control/fairino_dual_moveit_config/config/fairino.urdf (robot description, URDF)
Before this commit: robot dual_robot, 20 links, 19 joints
Links:
- link robot1_base_link: mass 1.6231 -> 1.6185; geometry collision mesh filename=file://$(find fairino_description)/meshes/fairino5_v6/base_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; visual mesh filename=file://$(find fairino_description)/meshes/fairino5_v6/base_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
- link robot1_forearm_link: mass 2.9964 -> 7.6737; geometry collision mesh filename=file://$(find fairino_description)/meshes/fairino5_v6/forea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; visual mesh filename=file://$(find fairino_description)/meshes/fairino5_v6/forea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
- link robot1_shoulder_link: mass 3.7152 -> 4.3771; geometry collision mesh filename=file://$(find fairino_description)/meshes/fairino5_v6/shoul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; visual mesh filename=file://$(find fairino_description)/meshes/fairino5_v6/shoul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
- link robot1_upperarm_link: mass 9.4622 -> 14.458; geometry collision mesh filename=file://$(find fairino_description)/meshes/fairino5_v6/upper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; visual mesh filename=file://$(find fairino_description)/meshes/fairino5_v6/upper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
- link robot1_wrist1_link: mass 2.1573 -> 1.6266; geometry collision mesh filename=file://$(find fairino_description)/meshes/fairino5_v6/wrist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; visual mesh filename=file://$(find fairino_description)/meshes/fairino5_v6/wrist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
- link robot1_wrist2_link: mass 2.1573 -> 1.5812; geometry collision mesh filename=file://$(find fairino_description)/meshes/fairino5_v6/wrist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; visual mesh filename=file://$(find fairino_description)/meshes/fairino5_v6/wrist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
- link robot1_wrist3_link: mass 0.20145 -> 0.52542; geometry collision mesh filename=file://$(find fairino_description)/meshes/fairino5_v6/wrist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; visual mesh filename=file://$(find fairino_description)/meshes/fairino5_v6/wrist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
- link robot2_base_link: mass 1.6185 -> 1.6231; geometry collision mesh filename=file://$(find fairino_description)/meshes/fairino16_v6/base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; visual mesh filename=file://$(find fairino_description)/meshes/fairino16_v6/base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
- link robot2_forearm_link: mass 7.6737 -> 2.9964; geometry collision mesh filename=file://$(find fairino_description)/meshes/fairino16_v6/fore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; visual mesh filename=file://$(find fairino_description)/meshes/fairino16_v6/fore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
- link robot2_shoulder_link: mass 4.3771 -> 3.7152; geometry collision mesh filename=file://$(find fairino_description)/meshes/fairino16_v6/shou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; visual mesh filename=file://$(find fairino_description)/meshes/fairino16_v6/shou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
- link robot2_upperarm_link: mass 14.458 -> 9.4622; geometry collision mesh filename=file://$(find fairino_description)/meshes/fairino16_v6/uppe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; visual mesh filename=file://$(find fairino_description)/meshes/fairino16_v6/uppe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
- link robot2_wrist1_link: mass 1.6266 -> 2.1573; geometry collision mesh filename=file://$(find fairino_description)/meshes/fairino16_v6/wris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; visual mesh filename=file://$(find fairino_description)/meshes/fairino16_v6/wris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
- link robot2_wrist2_link: mass 1.5812 -> 2.1573; geometry collision mesh filename=file://$(find fairino_description)/meshes/fairino16_v6/wris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; visual mesh filename=file://$(find fairino_description)/meshes/fairino16_v6/wris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
- link robot2_wrist3_link: mass 0.52542 -> 0.20145; geometry collision mesh filename=file://$(find fairino_description)/meshes/fairino16_v6/wris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; visual mesh filename=file://$(find fairino_description)/meshes/fairino16_v6/wris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
Joints:
- joint fixed1: child robot1_base_link -> robot2_base_link
- joint fixed2: child robot2_base_link -> robot1_base_link
- joint fixed3: parent robot1_wrist3_link -> robot2_wrist3_link
- joint fixed4: parent robot2_wrist3_link -> robot1_wrist3_link
- joint robot1_j2: origin xyz=0 0 0.18 rpy=1.5708 0 0 -> xyz=0 0 0.152 rpy=1.5708 0 0
- joint robot1_j3: origin xyz=-0.52 0 0 rpy=0 0 0 -> xyz=-0.425 0 0 rpy=0 0 0
- joint robot1_j4: origin xyz=-0.4 0 0 rpy=0 0 0 -> xyz=-0.39501 0 0 rpy=0 0 0
- joint robot1_j5: origin xyz=0 0 0.159 rpy=1.5708 0 0 -> xyz=0 0 0.1021 rpy=1.5708 0 0
- joint robot1_j6: origin xyz=0 0 0.114 rpy=-1.5708 0 0 -> xyz=0 0 0.102 rpy=-1.5708 0 0
- joint robot2_j2: origin xyz=0 0 0.152 rpy=1.5708 0 0 -> xyz=0 0 0.18 rpy=1.5708 0 0
- joint robot2_j3: origin xyz=-0.425 0 0 rpy=0 0 0 -> xyz=-0.52 0 0 rpy=0 0 0
- joint robot2_j4: origin xyz=-0.39501 0 0 rpy=0 0 0 -> xyz=-0.4 0 0 rpy=0 0 0
- joint robot2_j5: origin xyz=0 0 0.1021 rpy=1.5708 0 0 -> xyz=0 0 0.159 rpy=1.5708 0 0
- joint robot2_j6: origin xyz=0 0 0.102 rpy=-1.5708 0 0 -> xyz=0 0 0.114 rpy=-1.5708 0 0

File: src/moveit_control/fairino_dual_moveit_config/config/fairino_dual_robot_gazebo.xacro (robot description, xacro)
@@ -9,4 +9,40 @@
         <plugin>gazebo_ros2_control/GazeboSystem</plugin>
     </hardware>
+    <joint name="robot2_j1">
+        <command_interface name="position"/>
+        <state_interface name="position">
+            <param name="initial_value">0.0</param>
+        </state_interface>
+    </joint>
+    <joint name="robot2_j2">
+        <command_interface name="position"/>
+        <state_interface name="position">
+            <param name="initial_value">0.0</param>
+        </state_interface>
+    </joint>
+    <joint name="robot2_j3">
+        <command_interface name="position"/>
+        <state_interface name="position">
+            <param name="initial_value">0.0</param>
+        </state_interface>
+    </joint>
+    <joint name="robot2_j4">
+        <command_interface name="position"/>
+        <state_interface name="position">
+            <param name="initial_value">0.0</param>
+        </state_interface>
+    </joint>
+    <joint name="robot2_j5">
+        <command_interface name="position"/>
+        <state_interface name="position">
+            <param name="initial_value">0.0</param>
+        </state_interface>
+    </joint>
+    <joint name="robot2_j6">
+        <command_interface name="position"/>
+        <state_interface name="position">
+            <param name="initial_value">0.0</param>
+        </state_interface>
+    </joint>
     <joint name="robot1_j1">
         <command_interface name="position"/>
@@ -45,40 +81,4 @@
         </state_interface>
     </joint>
-    <joint name="robot2_j1">
-        <command_interface name="position"/>
-        <state_interface name="position">
-            <param name="initial_value">0.0</param>
-        </state_interface>
-    </joint>
-    <joint name="robot2_j2">
-        <command_interface name="position"/>
-        <state_interface name="position">
-            <param name="initial_value">0.0</param>
-        </state_interface>
-    </joint>
-    <joint name="robot2_j3">
-        <command_interface name="position"/>
-        <state_interface name="position">
-            <param name="initial_value">0.0</param>
-        </state_interface>
-    </joint>
-    <joint name="robot2_j4">
-        <command_interface name="position"/>
-        <state_interface name="position">
-            <param name="initial_value">0.0</param>
-        </state_interface>
-    </joint>
-    <joint name="robot2_j5">
-        <command_interface name="position"/>
-        <state_interface name="position">
-            <param name="initial_value">0.0</param>
-        </state_interface>
-    </joint>
-    <joint name="robot2_j6">
-        <command_interface name="position"/>
-        <state_interface name="position">
-            <param name="initial_value">0.0</param>
-        </state_interface>
-    </joint>
     </ros2_control>
     <gazebo>
