Commit message: rename robot 1 and 2

File: src/moveit_control/fairino_dual_moveit_config/config/fairino.urdf (robot description, URDF)
Before this commit: robot dual_robot, 20 links, 19 joints
Joints:
- joint fixed3: child end1 -> end2
- joint fixed4: child end2 -> end1

Commit message: add tcp

File: src/moveit_control/fairino_dual_moveit_config/config/fairino.urdf (robot description, URDF)
Before this commit: robot dual_robot, 20 links, 19 joints
Links:
- added link tcp1
- added link tcp2
Joints:
- added joint fixed5: type fixed, parent robot2_wrist3_link, child tcp2, origin xyz=-0.0 -0.0 0.106  rpy=0  0  0
- added joint fixed6: type fixed, parent robot1_wrist3_link, child tcp1, origin xyz=-0.0 -0.0 0.10 rpy=0.0 0.0  0.0

Commit message: 1-22 commit

File: src/moveit_control/fairino_dual_moveit_config/config/fairino.urdf (robot description, URDF)
Before this commit: robot dual_robot, 22 links, 21 joints
Joints:
- joint fixed1: origin xyz=0.162 0.202 -0.14 rpy=1.57  0.0  1.57 -> xyz=0.162 0.152 -0.14 rpy=1.57  0.0  1.57
- joint fixed2: origin xyz=-0.11406305  0.12505026 -0.140 rpy=0.0 -1.57  0.0 -> xyz=-0.09806305  0.06005026 -0.140 rpy=0.0 -1.57  0.0
- joint fixed3: origin xyz=-0.08 -0.06 0.23  rpy=0  1.57  0 -> xyz=-0.00 -0.00 0.11  rpy=0  0.0 3.14159
- joint fixed4: origin xyz=-0.05 -0.05 0.101 rpy=0.0 0.0  0.0 -> xyz=-0.00 -0.0 0.101 rpy=0.0 0.0 -0.785
- joint wall_fixed: origin xyz=0 0.8 0.2 rpy=-0.2 0 0 -> xyz=0 0.55 0.2 rpy=-0.261 0 0

Commit message: check servo bug

File: src/moveit_control/fairino_dual_moveit_config/config/fairino.urdf (robot description, URDF)
Before this commit: robot dual_robot, 22 links, 21 joints
Links:
- added link cube_link1, mass 1.0; collision box size=0.4 0.2 0.8; visual box size=0.4 0.2 0.8
- added link cube_link2, mass 1.0; collision box size=0.19 0.6 0.8; visual box size=0.19 0.6 0.8
- added link cube_link3, mass 1.0; collision box size=0.19 0.6 0.8; visual box size=0.19 0.6 0.8
Joints:
- added joint cube1_fixed: type fixed, parent base_dual_arm, child cube_link1, origin xyz=0.20 0.85 0.95 rpy=0 0 0
- added joint cube2_fixed: type fixed, parent wall, child cube_link2, origin xyz=-1.1 0 0.95 rpy=0 0 0
- added joint cube3_fixed: type fixed, parent wall, child cube_link3, origin xyz=1.1 0 0.95 rpy=0 0 0
- joint fixed1: origin xyz=0.162 0.152 -0.14 rpy=1.57  0.0  1.57 -> xyz=0.162 0.107 -0.14 rpy=1.57  0.785  1.57
- joint fixed4: origin xyz=-0.00 -0.0 0.101 rpy=0.0 0.0 -0.785 -> xyz=-0.00 -0.0 0.101 rpy=0.0 0.0 -3.14

Commit message: 0203

File: src/moveit_control/fairino_dual_moveit_config/config/fairino.urdf (robot description, URDF)
Before this commit: robot dual_robot, 25 links, 24 joints
Links:
- link cube_link1: geometry collision box size=0.5 0.2 0.8; visual box size=0.5 0.2 0.8
Joints:
- joint cube1_fixed: origin xyz=0.20 0.85 0.95 rpy=0 0 0 -> xyz=0.25 0.85 0.95 rpy=0 0 0
- joint robot1_j5: limit lower=-3.0543 upper=3.0543 effort=28 velocity=3.2 -> lower=-2.5543 upper=3.0543 effort=28 velocity=3.2

Commit message: 0303

File: src/moveit_control/fairino_dual_moveit_config/config/fairino.urdf (robot description, URDF)
Before this commit: robot dual_robot, 25 links, 24 joints
Joints:
- joint fixed4: origin xyz=-0.00 -0.0 0.101 rpy=0.0 0.0 -3.14 -> xyz=-0.00 -0.0 0.101 rpy=-3.14 0.0 0.0
